Commit message: robot description adjusted

File: robot_description/urdf/robot.xacro (robot description, xacro)
@@ -1,264 +1,252 @@
 <?xml version='1.0'?>
 <robot name="myrobot" xmlns:xacro="http://www.ros.org/wiki/xacro">
+  <xacro:property name="M_PI" value="3.1415926535897931" />
   <xacro:include filename="$(find robot_description)/urdf/robot.gazebo" />
   <xacro:include filename="$(find robot_description)/urdf/materials.xacro" />
+  <!-- <xacro:include filename="$(find robot_description)/urdf/macros.xacro"/> -->
   <!-- Base Robotic -->
   <link name="base_link">
     <inertial>
-      <mass value="2.0" />
+      <mass value="2" />
+      <origin xyz="0 0 0.0" />
+      <inertia ixx="0.01" ixy="0.0" ixz="0.0"
+        iyy="0.01" iyz="0.0" izz="0.5" />
+    </inertial>
+      <visual>
+        <origin xyz="0 0 0" rpy="0 0 0" />
+        <geometry>
+          <cylinder length="0.0095" radius="0.2245"/>
+        </geometry>
+        <material name ="White" />
+      </visual>
+      <collision>
+        <origin xyz="0 0 0" rpy="0 0 0" />
+        <geometry>
+          <cylinder length="0.0095" radius="0.2245"/>
+        </geometry>
+      </collision>
+  </link>
+  <!-- Bateria -->
+  <link name="battery_box">
+    <inertial>
+      <mass value="0.001" />
       <origin xyz="0 0 0" />
-      <inertia ixx="0.01" ixy="0.0" ixz="0.0"
-               iyy="0.01" iyz="0.0" izz="0.1" />
-    </inertial>
-    <visual>
-      <origin xyz="0 0 0" rpy="0 0 0" />
-      <geometry name="guntherbot_geom">
-        <mesh filename="$(find robot_description)/meshes/robot.stl" scale="0.01 0.01 0.01"/>
-      </geometry>
-      <material name="ChassisRed">
-        <color rgba="0.851 0.0 0.0 1.0"/>
-      </material>
-    </visual>
+      <inertia ixx="0.0001" ixy="0.0" ixz="0.0"
+        iyy="0.0001" iyz="0.0"
+        izz="0.0001" />
+    </inertial>
+      <visual>
+        <origin xyz="0 0 0" rpy="0 0 0" />
+        <geometry>
+          <box size="0.1778 0.3366 0.0762" />
+        </geometry>
+        <material name ="veryDarkGrey" />
+      </visual>
+      <collision>
+        <origin xyz="0 0 0" rpy="0 0 0" />
+        <geometry>
+          <box size="0.1778 0.3366 0.0762" />
+        </geometry>
+      </collision>
+  </link>
+  <joint name="battery_box_joint" type="fixed">
+    <origin xyz="0 0 -0.04285" rpy="0 0 0" />
+    <parent link="base_link" />
+    <child link="battery_box" />
+  </joint>
+  <!-- Roda Castor Frontal -->
+  <link name="front_caster">
+    <inertial>
+      <mass value="0.001" />
+      <origin xyz="0 0 0" />
+      <inertia ixx="0.0001" ixy="0.0" ixz="0.0"
+          iyy="0.0001" iyz="0.0"
+          izz="0.0001" />
+    </inertial>
+      <visual>
+        <origin xyz="0 0 0" rpy="-1.5707 0 1.5707" />
+        <geometry>
+          <mesh filename="package://robot_description/meshes/castor.dae"/>
+        </geometry>
+        <material name ="light_grey">
+          <color rgba="0.6 0.6 0.6 1"/>
+        </material>
+      </visual>
+      <collision>
+        <origin xyz="0 0 0" rpy="-1.5707 0 1.5707" />
+        <geometry>
+          <cylinder length="0.0605" radius="0.097"/>
+        </geometry>
+      </collision>
+  </link>
+  <joint name="front_caster_joint" type="fixed">
+    <origin xyz="0.18745 0 -0.00475" rpy="0 0 0" />
+    <parent link="base_link" />
+    <child link="front_caster" />
+  </joint>
+  <link name="rear_caster">
+    <inertial>
+      <mass value="0.001" />
+      <origin xyz="0 0 0" />
+      <inertia ixx="0.0001" ixy="0.0" ixz="0.0"
+        iyy="0.0001" iyz="0.0"
+        izz="0.0001" />
+      </inertial>
+      <visual>
+        <origin xyz="0 0 0" rpy="-1.5707 0 1.5707" />
+        <geometry>
+          <mesh filename="package://robot_description/meshes/castor.dae"/>
+        </geometry>
+        <material name ="light_grey">
+          <color rgba="0.6 0.6 0.6 1"/>
+        </material>
+      </visual>
+      <collision>
+        <origin xyz="0 0 0" rpy="-1.5707 0 1.5707" />
+        <geometry>
+          <cylinder length="0.0605" radius="0.097"/>
+        </geometry>
+      </collision>
+  </link>
+  <joint name="rear_caster_joint" type="fixed">
+    <origin xyz="-0.18745 0 -0.00475" rpy="0 0 0" />
+    <parent link="base_link" />
+    <child link="rear_caster" />
+  </joint>
+  <link name="left_axle_link">
+    <inertial>
+      <origin xyz="0 0 0"/>
+      <mass value="0.01" />
+      <inertia ixx="0.001" ixy="0.0" ixz="0.0"
+        iyy="0.001" iyz="0.0" izz="0.001" />
+      </inertial>
+      <visual>
+        <origin xyz="0 0 0" rpy="0 1.5707 1.5707" />
+        <geometry>
+          <cylinder radius="0.00635" length = "0.00635"/>
+        </geometry>
+        <material name ="light_grey" />
+      </visual>
+      <collision>
+        <origin xyz="0 0 0" rpy="0 1.5707 1.5707" />
+        <geometry>
+          <cylinder radius="0.00635" length = "0.00635"/>
+        </geometry>
+      </collision>
+  </link>
+  <joint name="left_axle_joint" type="fixed">
+    <origin xyz="0 0.171475 0.017" rpy="0 0 0"/>
+    <parent link="battery_box"/>
+    <child link="left_axle_link"/>
+    <axis xyz="0 1 0"/>
+  </joint>
+  <link name="right_axle_link">
+    <inertial>
+      <origin xyz="0 0 0"/>
+      <mass value="0.01" />
+      <inertia ixx="0.001" ixy="0.0" ixz="0.0"
+        iyy="0.001" iyz="0.0" izz="0.001" />
+      </inertial>
+      <visual>
+        <origin xyz="0 0 0" rpy="0 1.5707 1.5707" />
+        <geometry>
+          <cylinder radius="0.00635" length = "0.00635"/>
+        </geometry>
+        <material name ="light_grey" />
+      </visual>
+      <collision>
+        <origin xyz="0 0 0" rpy="0 1.5707 1.5707" />
+        <geometry>
+          <cylinder radius="0.00635" length = "0.00635"/>
+        </geometry>
+      </collision>
+  </link>
+  <joint name="right_axle_joint" type="fixed">
+    <origin xyz="0 -0.171475 0.017" rpy="0 0 0"/>
+    <parent link="battery_box"/>
+    <child link="right_axle_link"/>
+    <axis xyz="0 1 0"/>
+  </joint>
+  <link name="left_wheel_link">
+    <inertial>
+      <origin xyz="0 0 0"/>
+      <mass value="0.01" />
+      <inertia ixx="0.001" ixy="0.0" ixz="0.0"
+        iyy="0.001" iyz="0.0" izz="0.001" />
+      </inertial>
+      <visual>
+        <origin xyz="0 0 0" rpy="0 1.5707 1.5707" />
+        <geometry>
+          <cylinder radius="0.0762" length = "0.03175"/>
+        </geometry>
+        <material name ="grey" />
+      </visual>
+      <collision>
+        <origin xyz="0 0 0" rpy="0 1.5707 1.5707" />
+        <geometry>
+          <cylinder radius="0.076" length = "0.03175"/>
+        </geometry>
+      </collision>
+  </link>
+  <joint name="left_wheel_joint" type="continuous">
+    <origin xyz="0 0.01905 0" rpy="0 0 0"/>
+    <parent link="left_axle_link"/>
+    <child link="left_wheel_link"/>
+    <axis xyz="0 1 0"/>
+  </joint>
+  <link name="right_wheel_link">
+    <inertial>
+      <origin xyz="0 0 0"/>
+      <mass value="0.01" />
+      <inertia ixx="0.001" ixy="0.0" ixz="0.0"
+        iyy="0.001" iyz="0.0" izz="0.001" />
+      </inertial>
+      <visual>
+        <origin xyz="0 0 0" rpy="0 1.5707 1.5707" />
+        <geometry>
+          <cylinder radius="0.0762" length = "0.03175"/>
+        </geometry>
+        <material name ="grey" />
+      </visual>
+      <collision>
+        <origin xyz="0 0 0" rpy="0 1.5707 1.5707" />
+        <geometry>
+          <cylinder radius="0.076" length = "0.03175"/>
+        </geometry>
+      </collision>
+  </link>
+  <!-- Fixed because we never rotate it anyway, it is just for show -->
+  <!-- NOTE This may prevent gazebo from working with this model -->
+  <joint name="right_wheel_joint" type="continuous">
+    <origin xyz="0 -0.01905 0" rpy="0 0 0"/>
+    <parent link="right_axle_link"/>
+    <child link="right_wheel_link"/>
+    <axis xyz="0 1 0"/>
+  </joint>
+  <!-- Rplidar Laser -->
+  <link name="base_laser">
     <collision>
-      <origin xyz="0 0 0" rpy="0 0 0" />
+      <origin xyz="0 0 0" rpy="0 0 1"/>
       <geometry>
-        <mesh filename="$(find robot_description)/meshes/robot.stl" scale="0.01 0.01 0.01"/>
+        <box size="0.1 0.1 0.1"/>
       </geometry>
     </collision>
-  </link>
-  <!-- Castor Frontal -->
-  <link name="front_caster">
-    <inertial>
-      <mass value="0.5" />
-      <origin xyz="0 0 0" />
-      <inertia ixx="0.01" ixy="0.0" ixz="0.0"
-               iyy="0.01" iyz="0.0" izz="0.01" />
-    </inertial>
     <visual>
-      <origin xyz="0 0 0" rpy="0 0 0" />
+      <origin xyz="0 0 0.008" rpy="0 -${M_PI/2} ${M_PI}"/>
       <geometry>
-        <mesh filename="$(find robot_description)/meshes/castor_front.stl" scale="0.01 0.01 0.01"/>
-      </geometry>
-      <material name ="light_grey">
-        <color rgba="0.6 0.6 0.6 1"/>
-      </material>
-    </visual>
-    <collision>
-      <origin xyz="0 0 0" rpy="0 1.5707 0" />
-      <geometry>
-        <cylinder length="0.027026" radius="0.0381"/>
-      </geometry>
-    </collision>
-  </link>
-  <joint name="front_caster_joint" type="fixed">
-    <!-- <origin xyz="-0.1930 0.4134 -0.065" rpy="0 0 0" /> -->
-    <origin xyz="0 0.2488 -0.03627" rpy="0 0 0" />
-    <parent link="base_link" />
-    <child link="front_caster" />
-  </joint>
-  <!-- Left Axle Link -->
-  <link name="left_axle_link">
-    <inertial>
-      <origin xyz="0 0 0"/>
-      <mass value="0.01" />
-      <inertia ixx="0.001" ixy="0.0" ixz="0.0"
-        iyy="0.001" iyz="0.0" izz="0.001" />
-    </inertial>
-    <visual>
-      <origin xyz="0 0 0" rpy="3.1414 1.5707 3.1414" />
-      <geometry>
-        <cylinder radius="0.00735" length = "0.0369"/>
-        <!-- 10.905 mm 0.01095*2 = 0.0219 m -->
-      </geometry>
-      <material name ="light_grey" />
-    </visual>
-    <collision>
-      <origin xyz="0 0 0" rpy="3.1414 1.5707 3.1414" />
-      <geometry>
-        <cylinder radius="0.00735" length = "0.0369"/>
-      </geometry>
-    </collision>
-  </link>
-  <joint name="left_axle_joint" type="fixed">
-    <origin xyz="-0.1675 0 0" rpy="3.1414 0 3.1415"/>
-    <parent link="base_link"/>
-    <child link="left_axle_link"/>
-    <axis xyz="0 1 0"/>
-  </joint>
-  <!-- Right Axle Link -->
-  <link name="right_axle_link">
-    <inertial>
-      <origin xyz="0 0 0"/>
-      <mass value="0.01" />
-      <inertia ixx="0.001" ixy="0.0" ixz="0.0"
-        iyy="0.001" iyz="0.0" izz="0.001" />
-    </inertial>
-    <visual>
-      <origin xyz="0 0 0" rpy="0 1.5707 0" />
-      <geometry>
-        <cylinder radius="0.00735" length = "0.0369"/>
-        <!-- 10.905 mm 0.01095*2 = 0.0219 m -->
-      </geometry>
-      <material name ="light_grey" />
-    </visual>
-    <collision>
-      <origin xyz="0 0 0" rpy="0 1.5707 0" />
-      <geometry>
-        <cylinder radius="0.00735" length = "0.0369"/>
-      </geometry>
-    </collision>
-  </link>
-  <joint name="right_axle_joint" type="fixed">
-    <origin xyz="0.1675 0 0" rpy="0 0 0"/>
-    <parent link="base_link"/>
-    <child link="right_axle_link"/>
-    <axis xyz="0 1 0"/>
-  </joint>
-  <!-- Left Wheel Link -->
-  <link name="left_wheel_link">
-    <inertial>
-      <origin xyz="0 0 0"/>
-      <mass value="0.5"/>
-      <inertia
-      ixx="0.001" ixy="0.0" ixz="0.0"
-      iyy="0.001" iyz="0.0"
-      izz="0.001"/>
-    </inertial>
-    <visual>
-      <origin xyz="0 0 0" rpy="0 0 0"/>
-      <geometry>
-        <mesh filename="$(find robot_description)/meshes/wheel.stl" scale="0.01 0.01 0.01"/>
-        <!-- <cylinder length="0.033" radius="0.076250"/> -->
-      </geometry>
-      <material name ="black" />
-    </visual>
-    <collision>
-      <origin xyz="0 0 0" rpy="0 1.5707 0" />
-      <geometry>
-        <cylinder length="0.033" radius="0.076250"/>
-      </geometry>
-    </collision>
-  </link>
-  <joint name="left_wheel_joint" type="continuous">
-    <!-- pi/2(90) = 1.5707     pi(180) = 3.1414 -->
-    <origin xyz="0.03895 0 0" rpy="0 0 0"/>
-    <!-- 20.5 mm 0.0205  r/2 = 0.01845-->
-    <parent link="left_axle_link"/>
-    <child link="left_wheel_link"/>
-    <axis xyz="1 0 0"/>
-  </joint>
-  <!-- Right Wheel Link -->
-  <link name="right_wheel_link">
-    <inertial>
-      <origin xyz="0 0 0"/>
-      <mass value="0.5"/>
-      <inertia
-      ixx="0.001" ixy="0.0" ixz="0.0"
-      iyy="0.001" iyz="0.0"
-      izz="0.001"/>
-    </inertial>
-    <visual>
-      <origin xyz="0 0 0" rpy="0 0 0"/>
-      <geometry>
-        <mesh filename="$(find robot_description)/meshes/wheel.stl" scale="0.01 0.01 0.01"/>
-        <!-- <cylinder length="0.033" radius="0.076250"/> -->
-      </geometry>
-      <material name ="black" />
-    </visual>
-    <collision>
-      <origin xyz="0 0 0" rpy="0 1.5707 0" />
-      <geometry>
-        <cylinder length="0.033" radius="0.076250"/>
-      </geometry>
-    </collision>
-  </link>
-  <joint name="right_wheel_joint" type="continuous">
-    <!-- pi = 1.5707     2pi = 3.1415 -->
-    <origin xyz="0.03895 0 0" rpy="0 0 0"/>
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